File: explorers_pwb.sch (KiCad schematic (older format))
At the start: 44 parts, among them IC1 ATMEGA328-P, J1 USB_2, K1 CONN_3, P1 CONN_2, P2 CONN_2, P3 CONN_2, P4 CONN_8, P5 CONN_4, P6 CONN_8, U1 FT232RL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

Commit message: Added the 0.1uF cap to the dtr / reset line which is required to bring the board out of reset after programming. Also increased the board rev to 1.1
Signed-off-by: Dominic Baratta <dbaratta@buffalo.edu>
Parts:
- added C18: 0.1uF, symbol CSMALL
Connections:
- wire segments 186 -> 188
Other:
- moved on the sheet: R4
Changed lines of the file:
@@
-EESchema Schematic File Version 2  date 11/7/2013 10:24:31 PM
+EESchema Schematic File Version 2  date 12/25/2013 9:05:12 AM
 LIBS:power
 LIBS:device
@@
 LIBS:explorers_lib
 LIBS:INTERFACE_BOARD-LIB
-EELAYER 43  0
+LIBS:explorers_pwb-cache
+EELAYER 25  0
 EELAYER END
 $Descr A 11000 8500
@@
 Sheet 1 1
 Title ""
-Date "8 nov 2013"
+Date "25 dec 2013"
 Rev ""
 Comp ""
@@
 Comment4 ""
 $EndDescr
+Connection ~ 3350 5850
+Wire Wire Line
+	3350 5850 3350 5700
+Wire Wire Line
+	3350 5700 3700 5700
+Wire Wire Line
+	3750 5850 3600 5850
 Wire Wire Line
 	7100 1450 6800 1450
@@
 	3750 3350 3250 3350
 Wire Wire Line
-	4450 2900 4550 2900
-Wire Wire Line
-	4550 2900 4550 2800
+	4200 5700 4300 5700
+Wire Wire Line
+	4300 5700 4300 5600
 Wire Wire Line
 	4150 3100 3250 3100
@@
 	1200 6000 1200 6050
 Wire Wire Line
-	3950 2900 3950 3100
-Connection ~ 3950 3100
-Wire Wire Line
 	3250 3250 3750 3250
 Wire Wire Line
 	3550 5450 3250 5450
-Wire Wire Line
-	3550 5850 3250 5850
 Wire Wire Line
 	3250 6250 4000 6250
@@
 Wire Wire Line
 	6800 1550 7100 1550
+Wire Wire Line
+	3250 5850 3400 5850
+$Comp
+L CSMALL C18
+U 1 1 52BAE4A6
+P 3500 5850
+F 0 "C18" H 3525 5900 30  0000 L CNN
+F 1 "0.1uF" H 3525 5800 30  0000 L CNN
+	1    3500 5850
+	0    -1   -1   0
+$EndComp
 Text Label 6800 1950 0    45   ~ 0
 GPIO_6
@@
 NoConn ~ 3250 6550
 NoConn ~ 3250 6450
-Text GLabel 3550 5850 2    45   Input ~ 0
+Text GLabel 3750 5850 2    45   Input ~ 0
 RESET
 NoConn ~ 3250 6150
@@
 L +5V #PWR040
 U 1 1 52799C36
-P 4550 2800
-F 0 "#PWR040" H 4550 2890 20  0001 C CNN
-F 1 "+5V" H 4550 2890 30  0000 C CNN
-	1    4550 2800
+P 4300 5600
+F 0 "#PWR040" H 4300 5690 20  0001 C CNN
+F 1 "+5V" H 4300 5690 30  0000 C CNN
+	1    4300 5600
 	1    0    0    -1
 $EndComp
@@
 L R R4
 U 1 1 52799C1E
-P 4200 2900
-F 0 "R4" V 4280 2900 50  0000 C CNN
-F 1 "10k" V 4200 2900 50  0000 C CNN
-	1    4200 2900
+P 3950 5700
+F 0 "R4" V 4030 5700 50  0000 C CNN
+F 1 "10k" V 3950 5700 50  0000 C CNN
+	1    3950 5700
 	0    -1   -1   0
 $EndComp

Commit message: Final fix for the reset issue. Also generated new Gerber files.
Signed-off-by: Dominic Baratta <dbaratta@buffalo.edu>
Connections:
- wire segments 188 -> 187
